File: Battery_Buttons_V2.sch (EAGLE design)
At the start: 9 parts, among them U4 LP38693MP-3.3

Commit message: created new Battery package and added it to the PCB. I have also moved the switch around. Need to check for DRC errors etc
Parts:
- BAT1: device SparkFun-Electromechanical:BATTERY245PTH -> STM1061:BATTERY245PTH
Changed lines of the file:
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@@
 </classes>
 <parts>
-<part name="BAT1" library="SparkFun-Electromechanical" deviceset="BATTERY" device="245PTH">
+<part name="BAT1" library="STM1061" deviceset="BATTERY" device="245PTH">
 <attribute name="MF" value=""/>
 <attribute name="MPN" value=""/>
